File: hardware/openmote32_2_0_0/openmote32_2_0_0.sch (EAGLE design)
At the start: 39 parts, among them J1 XBEE_1-10, J2 XBEE_11-20, J3 JTAG_CONNECTOR, U1 AT86RF231, X1 16MHz

Commit message: Openmote v2 changes
Parts:
- removed B1: BALUNG-TYPE, WSNlib:BALUNG-TYPE
- removed C2: 22p, SparkFun:CAP0402
- removed TP1, TP2, TP3, TP4, TP5, TP6: TESTPOINTSMALLEST, WSNlib:TESTPOINTSMALLEST
- added C17, C18: 8p DNP, SparkFun:CAP0402
- added R3: 0R DNP, rcl:R-US_R0402
- added R4, R5: 0R, rcl:R-US_R0402
- added R6, R7: 33, rcl:R-US_R0402
- added TP10, TP11, TP12, TP7, TP8, TP9: TESTPOINTSMALLEST, WSNlib:TESTPOINTSMALLEST
- added U$1: DNP, WSNlib:ANTENNA_W_GROUNDS
- added U$2: USB_CONNECTOR, WSNlib:USB_CONNECTOR
- added U3: 2450FB15L0001, WSNlib:2450FB15L0001
- J1: value XBEE_1-10 -> XBEE_1-10SMD; device WSNlib:XBEE_1-10 -> WSNlib:XBEE_1-10SMD
- J2: value XBEE_11-20 -> XBEE_11-20SMD; device WSNlib:XBEE_11-20 -> WSNlib:XBEE_11-20SMD
- R2: value 0R -> 0R DNP
Connections:
- new net N$12: A1.P$1, R4.1
- new net N$15: R3.1, U$1G$1.P$1
- new net N$17: C5.2, C6.2, R5.2, U1.AEVDD, U1.DEVDD
- new net N$18: R7.2, U$2.D-
- net 3.3V: now also LED1.A, LED2.A, LED3.A, LED4.A, R5.1; no longer C5.2, C6.2, U1.AEVDD, U1.DEVDD
- net DBG_FRAME: no longer TP1.P$1
- net DBG_FSM: no longer TP4.P$1
- net DBG_ISR: no longer TP6.P$1
- net DBG_RADIO: no longer TP3.P$1
- net DBG_SLOT: no longer TP2.P$1
- net DBG_TASK: no longer TP5.P$1
- net GND: now also C1.1, C17.1, C18.1, TP10.P$1, TP11.P$1, TP12.P$1, TP7.P$1, TP8.P$1, TP9.P$1, U$1G$2.GND, U$1G$3.GND, U$1G$4.GND, U$1G$5.GND, U$2.GND, U1.AVSS(PAD)1, U1.AVSS(PAD)2, U1.AVSS(PAD)3, U1.AVSS(PAD)4, U1.AVSS(PAD)5, U3.GND@1, U3.GND@2; no longer B1.GND_1, B1.GND_2, B1.NC, LED1.C, LED2.C, LED3.C, LED4.C
- net K20_USBDM: now also R7.1
- net K20_USBDP: now also R6.1
- net LED1: now also LED1.C; no longer LED1.A
- net LED2: now also LED2.C; no longer LED2.A
- net LED3: now also LED3.C; no longer LED3.A
- net LED4: now also LED4.C; no longer LED4.A
- net N$1: now also U1.RFP, U3.BAL2; no longer B1.RFN, C2.2
- net N$11: now also C17.2
- net N$2: now also U1.RFN, U3.BAL1; no longer B1.RFP, C1.2
- net N$3: now also R3.2, R4.2, U3.UNB; no longer A1.P$1, B1.RF_UNB
- net N$4: now also C1.2, U3.DCFEED; no longer C2.1, U1.RFN
- net N$5: now also R6.2, U$2.D+; no longer C1.1, U1.RFP
- net N$8: now also C18.2
Other:
- note removed: "Check if its OK"
- moved on the sheet: A1, C1, LED1, LED2, LED3, LED4
